File: esp32_mine.kicad_pcb (KiCad board)
At the start: 2 copper layers, 36 x 68.8 mm, 76 parts, among them J1 USB_C_Receptacle_USB2.0_14P, J2 Conn_01x02_Pin, J3 Conn_01x18_Pin, J5 Conn_01x18_Pin, Q1 AO3401A, U1 ESP32-S3, U2 W25Q128JVS, U3 MCP73831-2-OT, U4 AMS1117-3.3, Y1 32.768 kHz, Y2 40MHz(10ppm)

Commit message: Add files via upload
Parts:
- removed G***: LOGO, Library:logo
- added C1: 0.1uF, Capacitor_SMD:C_0402_1005Metric, F.Cu at (168.5, 94.8)
- added C12: 0.1uF, Capacitor_SMD:C_0402_1005Metric, F.Cu at (171.2, 101.0)
- added C5: 0.1uF, Capacitor_SMD:C_0402_1005Metric, F.Cu at (169.0, 96.8)
- added C9: 0.1uF, Capacitor_SMD:C_0402_1005Metric, F.Cu at (169.2, 98.2)
- added J4: Conn_01x02_Pin, Connector_PinSocket_2.54mm:PinSocket_1x02_P2.54mm_Vertical, F.Cu at (168.5, 101.5)
- added Rm1: 0R, Resistor_SMD:R_0402_1005Metric, F.Cu at (161.0, 93.8)
- added Rm2: 0R, Resistor_SMD:R_0402_1005Metric, F.Cu at (158.8, 94.2)
- added Rm3: 0R, Resistor_SMD:R_0402_1005Metric, F.Cu at (164.8, 100.0)
- added U5: MPU-6050, mpu:QFN50P400X400X95-24N, F.Cu at (164.8, 95.2)
- added _: LOGO, aizeronix logo:aizeronix, F.Cu at (174.8, 105.2)
Routing:
- net IO17/SCL: track 33.3 -> 100.8 mm, vias 3 -> 5
- net IO18/SDA: track 34.2 -> 91.3 mm, vias 3 -> 6
- net VDD_CPU: track 121.1 -> 152.0 mm, vias 7 -> 11
- net INT: track 0.00 -> 9.67 mm, vias 0 -> 2
- net Net-(C1-Pad2): track 0.00 -> 7.11 mm
- net Net-(U5-REGOUT): track 0.00 -> 4.51 mm
- net Net-(U5-CPOUT): track 0.00 -> 4.30 mm
- net AD0: track 0.00 -> 3.09 mm
- net XCL: track 0.00 -> 2.63 mm
- net GND: track 14.6 -> 17.0 mm
- net XDA: track 0.00 -> 2.07 mm, vias 0 -> 1
- net Net-(U5-VDD): track 0.00 -> 1.90 mm
- net unconnected-(U5-RESV-Pad22): track 0.00 -> 1.63 mm
- net unconnected-(U5-RESV-Pad21): track 0.00 -> 1.63 mm
- net unconnected-(U5-CLKIN-Pad1): track 0.00 -> 1.57 mm
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