File: esp32_mine.kicad_sch (KiCad schematic)
At the start: 75 parts, among them J1 USB_C_Receptacle_USB2.0_14P, J2 Conn_01x02_Pin, J3 Conn_01x18_Pin, J5 Conn_01x18_Pin, Q1 AO3401A, U1 ESP32-S3, U2 W25Q128JVS, U3 MCP73831-2-OT, U4 AMS1117-3.3, Y1 32.768 kHz, Y2 40MHz(10ppm)

Commit message: Add files via upload
Parts:
- added C1, C12, C5, C9: 0.1uF, Capacitor_SMD:C_0402_1005Metric, symbol Device:C
- added J4: Conn_01x02_Pin, Connector_PinSocket_2.54mm:PinSocket_1x02_P2.54mm_Vertical, symbol Connector:Conn_01x02_Pin
- added Rm1, Rm2, Rm3: 0R, Resistor_SMD:R_0402_1005Metric, symbol Device:R
- added U5: MPU-6050, mpu:QFN50P400X400X95-24N, symbol mpu:MPU-6050
Connections:
- net +3V3: now also C12.1, Rm1.2, Rm2.2, U5.8 (VLOGIC)
- net GND: now also C9.2, Rm3.1, U5.11 (FSYNC), U5.18 (GND)
- net IO17/SCL: now also J4.2 (Pin_2), Rm1.1, U5.23 (SCL)
- net IO18/SDA: now also J4.1 (Pin_1), Rm2.1, U5.24 (SDA)
- new net: C1.2, C12.2, C5.2
- new net: C1.1, U5.20 (CPOUT)
- new net: C9.1, U5.10 (REGOUT)
- new net: C5.1, U5.13 (VDD)
- new net: U5.14 (NC), U5.15 (NC), U5.16 (NC), U5.17 (NC), U5.2 (NC), U5.3 (NC), U5.4 (NC), U5.5 (NC)
- new net: U5.19 (RESV), U5.21 (RESV), U5.22 (RESV)
- new net AD0: Rm3.2, U5.9 (AD0)
- new net INT: U5.12 (INT)
- new net XCL: U5.7 (AUX_CL)
- new net XDA: U5.6 (AUX_DA)
